Commit message: Feat: Configura MJCF para simulação com atuadores e ambiente
Adiciona atuadores de posição para o braço e a garra. Corrige o `ctrlrange` da GUI para corresponder aos limites das juntas em radianos.

Resolve o travamento da `shoulder_pan_joint` na inicialização, excluindo a colisão entre a base (`world`) e o ombro (`shoulder_link`).

O modelo agora inclui um chão (`floor`) e um cubo (`object_box`) para testes. A estrutura do XML foi otimizada com o uso de `default classes` e as restrições da garra foram configuradas com `<equality>`.

File: ur3_onrobot_rg2_model/ur3_onrobot_rg2.urdf.xacro (robot description, xacro)
@@ -57,5 +57,5 @@
       <origin rpy="0 0 3.141592653589793" xyz="0 0 0"/>
       <geometry>
-        <mesh filename="meshes/visual/base.stl"/>
+        <mesh filename="meshes/visual/v_base.stl"/>
       </geometry>
       <material name="LightGrey">
@@ -66,5 +66,5 @@
       <origin rpy="0 0 3.141592653589793" xyz="0 0 0"/>
       <geometry>
-        <mesh filename="meshes/collision/base.stl"/>
+        <mesh filename="meshes/collision/c_base.stl"/>
       </geometry>
     </collision>
@@ -87,5 +87,5 @@
       <origin rpy="0 0 3.141592653589793" xyz="0 0 0"/>
       <geometry>
-        <mesh filename="meshes/visual/shoulder.stl"/>
+        <mesh filename="meshes/visual/v_shoulder.stl"/>
       </geometry>
       <material name="LightGrey">
@@ -96,5 +96,5 @@
       <origin rpy="0 0 3.141592653589793" xyz="0 0 0"/>
       <geometry>
-        <mesh filename="meshes/collision/shoulder.stl"/>
+        <mesh filename="meshes/collision/c_shoulder.stl"/>
       </geometry>
     </collision>
@@ -117,5 +117,5 @@
       <origin rpy="1.5707963267948966 0 -1.5707963267948966" xyz="0 0 0.1198"/>
       <geometry>
-        <mesh filename="meshes/visual/upperarm.stl"/>
+        <mesh filename="meshes/visual/v_upperarm.stl"/>
       </geometry>
       <material name="LightGrey">
@@ -126,5 +126,5 @@
       <origin rpy="1.5707963267948966 0 -1.5707963267948966" xyz="0 0 0.1198"/>
       <geometry>
-        <mesh filename="meshes/collision/upperarm.stl"/>
+        <mesh filename="meshes/collision/c_upperarm.stl"/>
       </geometry>
     </collision>
@@ -147,5 +147,5 @@
       <origin rpy="1.5707963267948966 0 -1.5707963267948966" xyz="0 0 0.0275"/>
       <geometry>
-        <mesh filename="meshes/visual/forearm.stl"/>
+        <mesh filename="meshes/visual/v_forearm.stl"/>
       </geometry>
       <material name="LightGrey">
@@ -156,5 +156,5 @@
       <origin rpy="1.5707963267948966 0 -1.5707963267948966" xyz="0 0 0.0275"/>
       <geometry>
-        <mesh filename="meshes/collision/forearm.stl"/>
+        <mesh filename="meshes/collision/c_forearm.stl"/>
       </geometry>
     </collision>
@@ -178,5 +178,5 @@
       <origin rpy="1.5707963267948966 0 0" xyz="0 0 -0.085"/>
       <geometry>
-        <mesh filename="meshes/visual/wrist1.stl"/>
+        <mesh filename="meshes/visual/v_wrist1.stl"/>
       </geometry>
       <material name="LightGrey">
@@ -187,5 +187,5 @@
       <origin rpy="1.5707963267948966 0 0" xyz="0 0 -0.085"/>
       <geometry>
-        <mesh filename="meshes/collision/wrist1.stl"/>
+        <mesh filename="meshes/collision/c_wrist1.stl"/>
       </geometry>
     </collision>
@@ -208,5 +208,5 @@
       <origin rpy="0 0 0" xyz="0 0 -0.083"/>
       <geometry>
-        <mesh filename="meshes/visual/wrist2.stl"/>
+        <mesh filename="meshes/visual/v_wrist2.stl"/>
       </geometry>
       <material name="LightGrey">
@@ -217,5 +217,5 @@
       <origin rpy="0 0 0" xyz="0 0 -0.083"/>
       <geometry>
-        <mesh filename="meshes/collision/wrist2.stl"/>
+        <mesh filename="meshes/collision/c_wrist2.stl"/>
       </geometry>
     </collision>
@@ -238,5 +238,5 @@
       <origin rpy="1.5707963267948966 0 0" xyz="0 -0.00255 -0.082"/>
       <geometry>
-        <mesh filename="meshes/visual/wrist3.stl"/>
+        <mesh filename="meshes/visual/v_wrist3.stl"/>
       </geometry>
       <material name="LightGrey">
@@ -247,5 +247,5 @@
       <origin rpy="1.5707963267948966 0 0" xyz="0 -0.00255 -0.082"/>
       <geometry>
-        <mesh filename="meshes/collision/wrist3.stl"/>
+        <mesh filename="meshes/collision/c_wrist3.stl"/>
       </geometry>
     </collision>
@@ -306,5 +306,5 @@
       <origin rpy="0 0 0" xyz="0 0 0"/>
       <geometry>
-        <mesh filename="meshes/visual/base_link.stl"/>
+        <mesh filename="meshes/visual/v_base_link.stl"/>
       </geometry>
       <material name="">
@@ -315,5 +315,5 @@
       <origin rpy="0 0 0" xyz="0 0 0"/>
       <geometry>
-        <mesh filename="meshes/collision/base_link.stl"/>
+        <mesh filename="meshes/collision/c_base_link.stl"/>
       </geometry>
     </collision>
@@ -328,5 +328,5 @@
       <origin rpy="0 0 0" xyz="0 0 0"/>
       <geometry>
-        <mesh filename="meshes/visual/outer_knuckle.stl"/>
+        <mesh filename="meshes/visual/v_outer_knuckle.stl"/>
       </geometry>
       <material name="">
@@ -337,5 +337,5 @@
       <origin rpy="0 0 0" xyz="0 0 0"/>
       <geometry>
-        <mesh filename="meshes/collision/outer_knuckle.stl"/>
+        <mesh filename="meshes/collision/c_outer_knuckle.stl"/>
       </geometry>
     </collision>
@@ -350,5 +350,5 @@
       <origin rpy="0 0 0" xyz="0 0 0"/>
       <geometry>
-        <mesh filename="meshes/visual/inner_knuckle.stl"/>
+        <mesh filename="meshes/visual/v_inner_knuckle.stl"/>
       </geometry>
       <material name="">
@@ -359,5 +359,5 @@
       <origin rpy="0 0 0" xyz="0 0 0"/>
       <geometry>
-        <mesh filename="meshes/collision/inner_knuckle.stl"/>
+        <mesh filename="meshes/collision/c_inner_knuckle.stl"/>
       </geometry>
     </collision>
@@ -372,5 +372,5 @@
       <origin rpy="0 0 0" xyz="0 0 0"/>
       <geometry>
-        <mesh filename="meshes/visual/inner_finger.stl"/>
+        <mesh filename="meshes/visual/v_inner_finger.stl"/>
       </geometry>
       <material name="">
@@ -381,5 +381,5 @@
       <origin rpy="0 0 0" xyz="0 0 0"/>
       <geometry>
-        <mesh filename="meshes/collision/inner_finger.stl"/>
+        <mesh filename="meshes/collision/c_inner_finger.stl"/>
       </geometry>
     </collision>
@@ -394,5 +394,5 @@
       <origin rpy="0 0 0" xyz="0 0 0"/>
       <geometry>
-        <mesh filename="meshes/visual/outer_knuckle.stl"/>
+        <mesh filename="meshes/visual/v_outer_knuckle.stl"/>
       </geometry>
       <material name="">
@@ -403,5 +403,5 @@
       <origin rpy="0 0 0" xyz="0 0 0"/>
       <geometry>
-        <mesh filename="meshes/collision/outer_knuckle.stl"/>
+        <mesh filename="meshes/collision/c_outer_knuckle.stl"/>
       </geometry>
     </collision>
@@ -416,5 +416,5 @@
       <origin rpy="0 0 0" xyz="0 0 0"/>
       <geometry>
-        <mesh filename="meshes/visual/inner_knuckle.stl"/>
+        <mesh filename="meshes/visual/v_inner_knuckle.stl"/>
       </geometry>
       <material name="">
@@ -425,5 +425,5 @@
       <origin rpy="0 0 0" xyz="0 0 0"/>
       <geometry>
-        <mesh filename="meshes/collision/inner_knuckle.stl"/>
+        <mesh filename="meshes/collision/c_inner_knuckle.stl"/>
       </geometry>
     </collision>
@@ -438,5 +438,5 @@
       <origin rpy="0 0 0" xyz="0 0 0"/>
       <geometry>
-        <mesh filename="meshes/visual/inner_finger.stl"/>
+        <mesh filename="meshes/visual/v_inner_finger.stl"/>
       </geometry>
       <material name="">
@@ -447,5 +447,5 @@
       <origin rpy="0 0 0" xyz="0 0 0"/>
       <geometry>
-        <mesh filename="meshes/collision/inner_finger.stl"/>
+        <mesh filename="meshes/collision/c_inner_finger.stl"/>
       </geometry>
     </collision>
